Commit message: Add control tunning

File: zeabus_description/urdf/pelican_sensors.urdf.xacro (robot description, xacro)
@@ -127,4 +127,5 @@
       <child link="gx4_45_imu_link"/>
       <origin xyz="0 0 0" rpy="-1.59523 0 3.141593"/>
+      <!--<origin xyz="0 0 0" rpy="-M_PI/2 0 M_PI"/>-->
    </joint>
    <link name="gx4_45_imu_link">

Commit message: commit 19/06/17

File: zeabus_description/urdf/pelican_sensors.urdf.xacro (robot description, xacro)
@@ -126,5 +126,5 @@
       <parent link="base_link"/>
       <child link="gx4_45_imu_link"/>
-      <origin xyz="0 0 0" rpy="-1.59523 0 3.141593"/>
+      <origin xyz="0 0 0" rpy="-1.5743 0.013 3.141593"/>
       <!--<origin xyz="0 0 0" rpy="-M_PI/2 0 M_PI"/>-->
    </joint>

Commit message: using pressure sensor to calculate z - axis

File: zeabus_description/urdf/pelican_sensors.urdf.xacro (robot description, xacro)
@@ -126,6 +126,5 @@
       <parent link="base_link"/>
       <child link="gx4_45_imu_link"/>
-      <origin xyz="0 0 0" rpy="-1.5743 0.013 3.141593"/>
-      <!--<origin xyz="0 0 0" rpy="-M_PI/2 0 M_PI"/>-->
+      <origin xyz="0 0 0" rpy="-1.5761 0.0183 3.141593"/>
    </joint>
    <link name="gx4_45_imu_link">

Commit message: commit at 3/7/17

File: zeabus_description/urdf/pelican_sensors.urdf.xacro (robot description, xacro)
@@ -126,5 +126,5 @@
       <parent link="base_link"/>
       <child link="gx4_45_imu_link"/>
-      <origin xyz="0 0 0" rpy="-1.5761 0.0183 3.141593"/>
+      <origin xyz="-0.2 -0.05 0" rpy="-1.5761 0.0183 3.141593"/>
    </joint>
    <link name="gx4_45_imu_link">
